Commit message: update xml + cyclone

File: ros2_ws/src/dev/description/properties/core.xacro (robot description, xacro)
@@ -4,28 +4,28 @@
   <!-- ================== Chassis ================== -->
   <!-- ========= Dimensions ========= -->
-  <xacro:property name="chassis_size_x" value="0.3" />
-  <xacro:property name="chassis_size_y" value="0.3" />
-  <xacro:property name="chassis_size_z" value="0.15" />
+  <xacro:property name="chassis_size_x" value="0.353" />
+  <xacro:property name="chassis_size_y" value="0.350" />
+  <xacro:property name="chassis_size_z" value="0.090" />
   <!-- ========= Origin ========= -->
-  <xacro:property name="chassis_to_origin_offset_x" value="${chassis_size_x / 2}" />
+  <xacro:property name="chassis_to_origin_offset_x" value="0" />
   <xacro:property name="chassis_to_origin_offset_y" value="0" />
-  <xacro:property name="chassis_to_origin_offset_z" value="${chassis_size_z / 2}" />
+  <xacro:property name="chassis_to_origin_offset_z" value="0" />
   <!-- ========= Joint offsets ========= -->
-  <xacro:property name="base_to_chassis_joint_x" value="-0.1" />
+  <xacro:property name="base_to_chassis_joint_x" value="0" />
   <xacro:property name="base_to_chassis_joint_y" value="0" />
-  <xacro:property name="base_to_chassis_joint_z" value="0" />
+  <xacro:property name="base_to_chassis_joint_z" value="0.035" />
   <!-- ========= Material ========= -->
   <xacro:property name="chassis_material" value="white" />
   <!-- ========= Inertial ========= -->
-  <xacro:property name="chassis_mass" value="0.5" />
+  <xacro:property name="chassis_mass" value="2.0" />
   <!-- ========= Gazebo ========= -->
   <xacro:property name="chassis_gazebo_material" value="Gazebo/White" />
   <!-- ================== Left wheel ================== -->
   <!-- ========= Dimensions ========= -->
-  <xacro:property name="left_wheel_size_xy" value="0.05" />
-  <xacro:property name="left_wheel_size_z" value="0.04" />
+  <xacro:property name="left_wheel_size_xy" value="0.07" />
+  <xacro:property name="left_wheel_size_z" value="0.014" />
   <!-- ========= Joint offsets ========= -->
   <xacro:property name="base_to_left_wheel_joint_x" value="0" />
-  <xacro:property name="base_to_left_wheel_joint_y" value="0.175" />
+  <xacro:property name="base_to_left_wheel_joint_y" value="0.1186" />
   <xacro:property name="base_to_left_wheel_joint_z" value="0" />
   <xacro:property name="base_to_left_wheel_joint_roll" value="${-pi / 2}" />
@@ -65,7 +65,7 @@
   <!-- ================== Caster wheel ================== -->
   <!-- ========= Dimensions ========= -->
-  <xacro:property name="caster_wheel_size_xyz" value="0.05" />
+  <xacro:property name="caster_wheel_size_xyz" value="0.07" />
   <!-- ========= Joint offsets ========= -->
-  <xacro:property name="base_to_caster_wheel_joint_x" value="0.24" />
+  <xacro:property name="base_to_caster_wheel_joint_x" value="0.154" />
   <xacro:property name="base_to_caster_wheel_joint_y" value="0" />
   <xacro:property name="base_to_caster_wheel_joint_z" value="0" />

File: ros2_ws/src/dev/description/properties/lidar.xacro (robot description, xacro)
@@ -4,14 +4,14 @@
   <!-- ================== Laser ================== -->
   <!-- ========= Dimensions ========= -->
-  <xacro:property name="laser_frame_size_xy" value="0.05" />
+  <xacro:property name="laser_frame_size_xy" value="0.07" />
   <xacro:property name="laser_frame_size_z" value="0.04" />
   <!-- ========= Joint offsets ========= -->
-  <xacro:property name="chassis_to_laser_frame_joint_x" value="0.15" />
+  <xacro:property name="chassis_to_laser_frame_joint_x" value="0.0311" />
   <xacro:property name="chassis_to_laser_frame_joint_y" value="0" />
-  <xacro:property name="chassis_to_laser_frame_joint_z" value="0.17" />
+  <xacro:property name="chassis_to_laser_frame_joint_z" value="0.075" />
   <!-- ========= Material ========= -->
   <xacro:property name="laser_frame_material" value="orange" />
   <!-- ========= Inertial ========= -->
-  <xacro:property name="laser_frame_mass" value="0.5" />
+  <xacro:property name="laser_frame_mass" value="0.3" />
   <!-- ========= Gazebo ========= -->
   <xacro:property name="laser_frame_gazebo_material" value="Gazebo/Orange" />

File: ros2_ws/src/dev/description/robot/core.xacro (robot description, xacro)
@@ -141,5 +141,5 @@
   <!-- ========= Joint ========= -->
   <joint name="caster_wheel_joint" type="fixed">
-    <parent link="chassis" />
+    <parent link="base_link" />
     <child link="caster_wheel" />
     <origin xyz="${base_to_caster_wheel_joint_x} ${base_to_caster_wheel_joint_y} ${base_to_caster_wheel_joint_z}" />
